File: GaussSpeedway.kicad_pcb (KiCad board)
At the start: 4 copper layers, 212.5 x 152.5 mm, 48 parts, among them J1 Barrel_Jack_Switch, J2 JST PH, T1 LinearTouch4, T2 Conn_01x01, T3 LinearTouch4, U1 STM32F051C6Tx, U2 MCP1754S-3302xCB, U3 ZXBM5210-SP, U4 ZXBM5210-SP, U5 ZXBM5210-SP

Commit message: up
Routing:
- net (no net): track 0.00 -> 73.7 mm
- net /G1_P: track 1189.0 -> 1168.9 mm
